File: kicad/buttons/buttons.kicad_pcb (KiCad board)
At the start: 2 copper layers, 70 x 22 mm, 17 parts, among them J1 Conn_01x08_Pin, SW1 B3W-1000, SW2 B3W-1000, SW3 B3W-1000, SW4 B3W-1000, SW5 B3W-1000, SW6 B3W-1000

Commit message: WIP
Parts:
- J1: footprint Connector_PinHeader_2.54mm:PinHeader_1x08_P2.54mm_Vertical -> Connector_JST:JST_XH_S8B-XH-A_1x08_P2.50mm_Horizontal
- R1, R2, R3, R4, R5, R6: value R -> 10k
- moved R6 10.1 mm to (135.5, 92.0), turned to 180 degrees
- moved J1 1.69 mm to (101.7, 93.6), turned to 180 degrees
- moved R1 1.41 mm to (83.1, 108.8)
- moved R2 1.41 mm to (83.1, 105.3)
- moved R3 1.41 mm to (83.1, 101.8)
- moved R4 1.41 mm to (83.1, 98.3)
Connections:
- J1 pad 1: Net-(J1-Pin_1) -> /Btn1
- J1 pad 2: unconnected-(J1-Pin_2-Pad2) -> /Btn2
- J1 pad 3: /Btn6 -> /Btn3
- J1 pad 4: /Btn5 -> /Btn4
- J1 pad 5: /Btn4 -> /Btn5
- J1 pad 6: /Btn3 -> /Btn6
- J1 pad 7: /Btn2 -> unconnected-(J1-Pin_7-Pad7)
- J1 pad 8: /Btn1 -> /3.3V
- R1 pad 1: Net-(J1-Pin_1) -> /3.3V
- R2 pad 1: Net-(J1-Pin_1) -> /3.3V
- R3 pad 1: Net-(J1-Pin_1) -> /3.3V
- R4 pad 1: Net-(J1-Pin_1) -> /3.3V
- R5 pad 1: Net-(J1-Pin_1) -> /3.3V
- R6 pad 1: Net-(J1-Pin_1) -> /3.3V
Routing:
- net Net-(J1-Pin_1): track 92.1 -> 0.00 mm
- net /3.3V: track 0.00 -> 89.9 mm
- net /Btn3: track 51.3 -> 22.2 mm
- net /Btn1: track 43.2 -> 20.0 mm
- net /Btn2: track 24.0 -> 7.36 mm
- net /Btn5: track 30.9 -> 41.6 mm
- net /Btn6: track 60.1 -> 53.7 mm
- net Net-(R4-Pad2): track 19.3 -> 21.0 mm
- net /Btn4: track 23.9 -> 22.7 mm
- net Net-(R1-Pad2): track 14.8 -> 13.7 mm
- net Net-(R6-Pad2): track 12.0 -> 12.7 mm
