File: kicad/buttons/buttons.kicad_sch (KiCad schematic)
At the start: 13 parts, among them J1 Conn_01x08_Pin, SW1 SW_Push, SW2 SW_Push, SW3 SW_Push, SW4 SW_Push, SW5 SW_Push, SW6 SW_Push

Commit message: finish buttons board
Parts:
- removed R5, R6: R, Resistor_THT:R_Axial_DIN0207_L6.3mm_D2.5mm_P10.16mm_Horizontal, symbol Device:R
- removed SW1, SW2, SW3, SW4, SW5, SW6: SW_Push, symbol Switch:SW_Push
- added R1, R2: R, Resistor_THT:R_Axial_DIN0207_L6.3mm_D2.5mm_P10.16mm_Horizontal, symbol Device:R
- added U1, U2, U3, U4, U5, U6: B3U-1000P, B3U-1000P, symbol omron b3u:B3U-1000P
- J1: footprint (none) -> Connector_PinHeader_2.54mm:PinHeader_1x08_P2.54mm_Vertical
- R6: renamed from R1; footprint Resistor_THT:R_Box_L8.4mm_W2.5mm_P5.08mm -> Resistor_THT:R_Axial_DIN0207_L6.3mm_D2.5mm_P10.16mm_Horizontal
- renumbered R2 to R5
Connections:
- net Btn1: now also U1.2
- net Btn2: now also U2.2
- net Btn3: now also U3.2
- net Btn4: now also U4.2
- net Btn5: now also U5.2
- net Btn6: now also U6.2
- net at R6.2: now also U6.1
- net at J1.1 (Pin_1), R3.1, R4.1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: now also R1.1, R2.1
- net at R3.2: now also U3.1
- net at R4.2: now also U4.1
- net at R5.2: now also U5.1
- new net: R1.2, U1.1
- new net: R2.2, U2.1
Other:
- moved on the sheet: R5

Commit message: improve buttons board
Parts:
- removed U1, U2, U3, U4, U5, U6: B3U-1000P, B3U-1000P, symbol omron b3u:B3U-1000P
- added SW1, SW2, SW3, SW4, SW5, SW6: B3W-1000, SW_B3W-1000_OMR, symbol omron b3w:B3W-1000
Connections:
- net Btn1: now also SW1.2
- net Btn2: now also SW2.2
- net Btn3: now also SW3.2
- net Btn4: now also SW4.2
- net Btn5: now also SW5.2
- net Btn6: now also SW6.2
- net at R1.2: now also SW1.3
- net at R2.2: now also SW2.3
- net at R6.2: now also SW6.3
- net at R3.2: now also SW3.3
- net at R5.2: now also SW5.3
- net at R4.2: now also SW4.3
- no-connect marks 1 -> 13
