File: kicad/buttons/buttons.kicad_sch (KiCad schematic)
At the start: 13 parts, among them J1 Conn_01x08_Pin, SW1 B3W-1000, SW2 B3W-1000, SW3 B3W-1000, SW4 B3W-1000, SW5 B3W-1000, SW6 B3W-1000

Commit message: WIP
Parts:
- J1: footprint Connector_PinHeader_2.54mm:PinHeader_1x08_P2.54mm_Vertical -> Connector_JST:JST_XH_S8B-XH-A_1x08_P2.50mm_Horizontal
- R1, R2, R3, R4, R5, R6: value R -> 10k
- SW1, SW2, SW3, SW4, SW5, SW6: footprint SW_B3W-1000_OMR -> Omron:SW_B3W-1000_OMR
Connections:
- net Btn1: now also J1.1 (Pin_1); no longer J1.8 (Pin_8)
- net Btn2: now also J1.2 (Pin_2); no longer J1.7 (Pin_7)
- net Btn3: now also J1.3 (Pin_3); no longer J1.6 (Pin_6)
- net Btn4: now also J1.4 (Pin_4); no longer J1.5 (Pin_5)
- net Btn5: now also J1.5 (Pin_5); no longer J1.4 (Pin_4)
- net Btn6: now also J1.6 (Pin_6); no longer J1.3 (Pin_3)
- net 3.3V: now reaches R1.1, R2.1, R3.1, R4.1, R5.1, R6.1
- net 3.3V: now also J1.8 (Pin_8); no longer J1.1 (Pin_1)
Changed lines of the file:
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@@
+	)
+	(junction
+		(at 80.01 25.4)
+		(diameter 0)
+		(color 0 0 0 0)
+	)
+	(junction
+		(at 146.05 25.4)
+		(diameter 0)
+		(color 0 0 0 0)
+	)
+	(junction
+		(at 179.07 25.4)
+		(diameter 0)
+		(color 0 0 0 0)
 	)
 	(junction
@@
 		(color 0 0 0 0)
 	)
-	(junction
-		(at 80.01 25.4)
-		(diameter 0)
-		(color 0 0 0 0)
-	)
-	(junction
-		(at 146.05 25.4)
-		(diameter 0)
-		(color 0 0 0 0)
-	)
-	(junction
-		(at 179.07 25.4)
-		(diameter 0)
-		(color 0 0 0 0)
-	)
 	(no_connect
 		(at 113.03 77.47)
 	)
 	(no_connect
+		(at 25.4 90.17)
+	)
+	(no_connect
 		(at 49.53 36.83)
 	)
@@
 	(no_connect
 		(at 212.09 77.47)
-	)
-	(no_connect
-		(at 27.94 27.94)
 	)
 	(no_connect
@@
 	(wire
 		(pts
-			(xy 27.94 25.4) (xy 46.99 25.4)
+			(xy 25.4 25.4) (xy 46.99 25.4)
 		)
 		(stroke
@@
 		)
 	)
+	(label "Btn1"
+		(at 25.4 74.93 0)
+		(effects
+			(font
+				(size 1.27 1.27)
+			)
+			(justify left bottom)
+		)
+	)
+	(label "3.3V"
+		(at 25.4 92.71 0)
+		(effects
+			(font
+				(size 1.27 1.27)
+			)
+			(justify left bottom)
+		)
+	)
 	(label "Btn5"
-		(at 27.94 33.02 0)
+		(at 25.4 85.09 0)
 		(effects
 			(font
@@
 		)
 	)
-	(label "Btn1"
-		(at 27.94 43.18 0)
+	(label "3.3V"
+		(at 25.4 25.4 180)
 		(effects
 			(font
 				(size 1.27 1.27)
 			)
-			(justify left bottom)
+			(justify right bottom)
 		)
 	)
@@
 	)
 	(label "Btn2"
-		(at 27.94 40.64 0)
+		(at 25.4 77.47 0)
 		(effects
 			(font
@@
 		)
 	)
-	(label "Btn4"
-		(at 27.94 35.56 0)
+	(label "Btn6"
+		(at 25.4 87.63 0)
 		(effects
 			(font
@@
 		)
 	)
+	(label "Btn4"
+		(at 25.4 82.55 0)
+		(effects
+			(font
+				(size 1.27 1.27)
+			)
+			(justify left bottom)
+		)
+	)
 	(label "Btn3"
-		(at 27.94 38.1 0)
+		(at 25.4 80.01 0)
 		(effects
 			(font
@@
 			)
 			(justify right bottom)
-		)
-	)
-	(label "Btn6"
-		(at 27.94 30.48 0)
-		(effects
-			(font
-				(size 1.27 1.27)
-			)
-			(justify left bottom)
 		)
 	)
@@
 			)
 		)
-		(property "Footprint" "SW_B3W-1000_OMR"
+		(property "Footprint" "Omron:SW_B3W-1000_OMR"
 			(at 82.55 36.83 0)
 			(hide yes)
@@
 			)
 		)
-		(property "Value" "R"
+		(property "Value" "10k"
 			(at 214.63 34.2899 0)
 			(show_name no)
@@
 				(path "/0e67d20b-756b-4fda-b523-6b8b59b452f1"
 					(reference "R1")
+					(unit 1)
+				)
+			)
+		)
+	)
+	(symbol
+		(lib_id "Connector:Conn_01x08_Pin")
+		(at 20.32 82.55 0)
+		(unit 1)
+		(body_style 1)
+		(exclude_from_sim no)
+		(in_bom yes)
+		(on_board yes)
+		(in_pos_files yes)
+		(dnp no)
+		(fields_autoplaced yes)
+		(property "Reference" "J1"
+			(at 20.955 69.85 0)
+			(show_name no)
+			(do_not_autoplace no)
+			(effects
+				(font
+					(size 1.27 1.27)
+				)
+			)
+		)
+		(property "Value" "Conn_01x08_Pin"
+			(at 20.955 72.39 0)
+			(show_name no)
+			(do_not_autoplace no)
+			(effects
+				(font
+					(size 1.27 1.27)
+				)
+			)
+		)
+		(property "Footprint" "Connector_JST:JST_XH_S8B-XH-A_1x08_P2.50mm_Horizontal"
+			(at 20.32 82.55 0)
+			(hide yes)
+			(show_name no)
+			(do_not_autoplace no)
+			(effects
+				(font
+					(size 1.27 1.27)
+				)
+			)
+		)
+		(property "Datasheet" ""
+			(at 20.32 82.55 0)
+			(hide yes)
+			(show_name no)
+			(do_not_autoplace no)
+			(effects
+				(font
+					(size 1.27 1.27)
+				)
+			)
+		)
+		(property "Description" "Generic connector, single row, 01x08, script generated"
+			(at 20.32 82.55 0)
+			(hide yes)
+			(show_name no)
+			(do_not_autoplace no)
+			(effects
+				(font
+					(size 1.27 1.27)
+				)
+			)
+		)
+		(pin "8"
+		)
+		(pin "2"
+		)
+		(pin "1"
+		)
+		(pin "3"
+		)
+		(pin "6"
+		)
+		(pin "5"
+		)
+		(pin "7"
+		)
+		(pin "4"
+		)
+		(instances
+			(project "buttons"
+				(path "/0e67d20b-756b-4fda-b523-6b8b59b452f1"
+					(reference "J1")
 					(unit 1)
 				)
@@
 			)
 		)
-		(property "Footprint" "SW_B3W-1000_OMR"
+		(property "Footprint" "Omron:SW_B3W-1000_OMR"
 			(at 49.53 36.83 0)
 			(hide yes)
@@
 			)
 		)
-		(property "Footprint" "SW_B3W-1000_OMR"
+		(property "Footprint" "Omron:SW_B3W-1000_OMR"
 			(at 181.61 36.83 0)
 			(hide yes)
@@
 			)
 		)
-		(property "Value" "R"
+		(property "Value" "10k"
 			(at 49.53 34.2899 0)
 			(show_name no)
@@
 			)
 		)
-		(property "Value" "R"
+		(property "Value" "10k"
 			(at 148.59 34.2899 0)
 			(show_name no)
@@
 			)
 		)
-		(property "Value" "R"
+		(property "Value" "10k"
 			(at 181.61 34.2899 0)
 			(show_name no)
@@
 			)
 		)
-		(property "Value" "R"
+		(property "Value" "10k"
 			(at 82.55 34.2899 0)
 			(show_name no)
@@
 			)
 		)
-		(property "Footprint" "SW_B3W-1000_OMR"
+		(property "Footprint" "Omron:SW_B3W-1000_OMR"
 			(at 115.57 36.83 0)
 			(hide yes)
@@
 			)
 		)
-		(property "Footprint" "SW_B3W-1000_OMR"
+		(property "Footprint" "Omron:SW_B3W-1000_OMR"
 			(at 214.63 36.83 0)
 			(hide yes)
@@
 			)
 		)
-		(property "Value" "R"
+		(property "Value" "10k"
 			(at 115.57 34.2899 0)
 			(show_name no)
@@
 			)
 		)
-		(property "Footprint" "SW_B3W-1000_OMR"
+		(property "Footprint" "Omron:SW_B3W-1000_OMR"
 			(at 148.59 36.83 0)
 			(hide yes)
@@
 					(unit 1)
 				)
-			)
-		)
-	)
-	(symbol
-		(lib_id "Connector:Conn_01x08_Pin")
-		(at 22.86 33.02 0)
-		(unit 1)
-		(body_style 1)
-		(exclude_from_sim no)
-		(in_bom yes)
-		(on_board yes)
-		(in_pos_files yes)
-		(dnp no)
-		(fields_autoplaced yes)
-		(property "Reference" "J1"
-			(at 23.495 20.32 0)
-			(show_name no)
-			(do_not_autoplace no)
-			(effects
-				(font
-					(size 1.27 1.27)
-				)
-			)
-		)
-		(property "Value" "Conn_01x08_Pin"
-			(at 23.495 22.86 0)
-			(show_name no)
-			(do_not_autoplace no)
-			(effects
-				(font
-					(size 1.27 1.27)
-				)
-			)
-		)
-		(property "Footprint" "Connector_PinHeader_2.54mm:PinHeader_1x08_P2.54mm_Vertical"
-			(at 22.86 33.02 0)
-			(hide yes)
-			(show_name no)
-			(do_not_autoplace no)
-			(effects
-				(font
-					(size 1.27 1.27)
-				)
-			)
-		)
-		(property "Datasheet" ""
-			(at 22.86 33.02 0)
-			(hide yes)
-			(show_name no)
-			(do_not_autoplace no)
-			(effects
-				(font
-					(size 1.27 1.27)
-				)
-			)
-		)
-		(property "Description" "Generic connector, single row, 01x08, script generated"
-			(at 22.86 33.02 0)
-			(hide yes)
-			(show_name no)
-			(do_not_autoplace no)
-			(effects
-				(font
-					(size 1.27 1.27)
-				)
-			)
-		)
-		(pin "8"
-		)
-		(pin "2"
-		)
-		(pin "1"
-		)
-		(pin "3"
-		)
-		(pin "6"
-		)
-		(pin "5"
-		)
-		(pin "7"
-		)
-		(pin "4"
-		)
-		(instances
-			(project "buttons"
-				(path "/0e67d20b-756b-4fda-b523-6b8b59b452f1"
-					(reference "J1")
-					(unit 1)
-				)
