File: kicad/hat/hat.kicad_pcb (KiCad board)
At the start: 2 copper layers, 65 x 36 mm, 17 parts, among them J1 GPIO, J2 FrontButtons, J3 DisplaySPI, J4 BatteryLevel, J5 PowerButton, J6 PowerWakeup

Commit message: WIP
Parts:
- removed BatteryVoltageDividerOnOffSwitch1: IRLF44N, Package_TO_SOT_THT:TO-220-3_Vertical
- removed DisplayOnOffSwitch1: IRLZ44N, Package_TO_SOT_THT:TO-220-3_Vertical
- moved C1 8.72 mm to (149.9, 69.2)
- moved C3 4.81 mm to (161.5, 68.7)
- moved C2 4.47 mm to (161.5, 71.7)
Connections:
- J1 pad 22: /DisplayOnOff -> /GPIO25
- J1 pad 33: /BatterNNP16 -> GND
- J1 pad 35: /BatteryVoltageDividerOnOff -> /GPIO19/PCM.FS
- R3 pad 1: /BatterNNP16 -> GND
Routing:
- net GND: track 89.9 -> 106.3 mm
- net /BatterNNP16: track 16.5 -> 0.00 mm
- net +5V: track 121.3 -> 129.3 mm
- net /SPI_GND: track 29.6 -> 37.1 mm
