File: kicad/power_on_button/power_on_button.kicad_pcb (KiCad board)
At the start: 2 copper layers, 23.2 x 24.1 mm, 6 parts, among them J1 Conn_01x02_Pin, SW1 B3W-1000

Commit message: wip
Parts:
- SW1: moved to B.Cu
- moved SW1 6.45 mm to (220.6, 107.5), turned to 0 degrees
Routing:
- net Net-(R1-Pad2): track 17.1 -> 23.6 mm
- net /Btn1: track 20.0 -> 24.7 mm

Commit message: add powert button to menu
Connections:
- J1 pad 1: /3.3V -> /Btn1
- J1 pad 2: /Btn1 -> /3.3V
Routing:
- net /Btn1: track 24.7 -> 7.48 mm
Changed lines of the file:
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@@
 			(remove_unused_layers no)
 			(roundrect_rratio 0.147059)
-			(net "/3.3V")
+			(net "/Btn1")
 			(pinfunction "Pin_1_1")
 			(pintype "passive")
@@
 			(layers "*.Cu" "*.Mask")
 			(remove_unused_layers no)
-			(net "/Btn1")
+			(net "/3.3V")
 			(pinfunction "Pin_2_2")
 			(pintype "passive")
@@
 	)
 	(segment
-		(start 229.75 109.65)
+		(start 232.25 109.05)
 		(end 231.3 108.1)
 		(width 0.2)
@@
 	)
 	(segment
-		(start 229.75 113.9)
-		(end 229.75 109.65)
+		(start 232.25 113.9)
+		(end 232.25 109.05)
 		(width 0.2)
 		(layer "B.Cu")
@@
 	)
 	(segment
-		(start 220.6 110.5)
-		(end 220.599998 110.499998)
+		(start 229.75 110.099999)
+		(end 227.150001 107.5)
 		(width 0.2)
 		(layer "B.Cu")
@@
 	)
 	(segment
-		(start 232.25 113.9)
-		(end 232.25 115.85)
+		(start 229.75 113.9)
+		(end 229.75 110.099999)
 		(width 0.2)
 		(layer "B.Cu")
-		(net "/Btn1")
-	)
-	(segment
-		(start 225.1 116.3)
-		(end 220.6 111.8)
-		(width 0.2)
-		(layer "B.Cu")
-		(net "/Btn1")
-	)
-	(segment
-		(start 232.25 115.85)
-		(end 231.8 116.3)
-		(width 0.2)
-		(layer "B.Cu")
-		(net "/Btn1")
-	)
-	(segment
-		(start 231.8 116.3)
-		(end 225.1 116.3)
-		(width 0.2)
-		(layer "B.Cu")
-		(net "/Btn1")
-	)
-	(segment
-		(start 220.6 111.8)
-		(end 220.6 110.5)
-		(width 0.2)
-		(layer "B.Cu")
-		(net "/Btn1")
-	)
-	(segment
-		(start 220.6 110.5)
-		(end 224.150001 110.5)
-		(width 0.2)
-		(layer "B.Cu")
-		(net "/Btn1")
-	)
-	(segment
-		(start 224.150001 110.5)
-		(end 227.150001 107.5)
-		(width 0.2)
-		(layer "B.Cu")

Commit message: fix bug in power on button routing in power on button
Connections:
- J1 pad 1: /Btn1 -> /GND
- J1 pad 2: /3.3V -> /BtnPower
- R1 pad 1: /3.3V -> /GND
- SW1 pad 2: /Btn1 -> /BtnPower
Routing:
- net /GND: track 0.00 -> 14.2 mm
- net /BtnPower: track 0.00 -> 8.51 mm
- net /Btn1: track 7.48 -> 0.00 mm
- net /3.3V: track 6.19 -> 0.00 mm
Changed lines of the file:
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@@
 			(remove_unused_layers no)
 			(roundrect_rratio 0.147059)
-			(net "/Btn1")
+			(net "/GND")
 			(pinfunction "Pin_1_1")
 			(pintype "passive")
@@
 			(layers "*.Cu" "*.Mask")
 			(remove_unused_layers no)
-			(net "/3.3V")
+			(net "/BtnPower")
 			(pinfunction "Pin_2_2")
 			(pintype "passive")
@@
 			(layers "*.Cu" "*.Mask")
 			(remove_unused_layers no)
-			(net "/3.3V")
+			(net "/GND")
 			(pintype "passive")
 		)
@@
 			(layers "*.Cu" "*.Mask")
 			(remove_unused_layers no)
-			(net "/Btn1")
+			(net "/BtnPower")
 			(pinfunction "2_2")
 			(pintype "unspecified")
@@
 	)
 	(segment
-		(start 232.25 109.05)
-		(end 231.3 108.1)
-		(width 0.2)
-		(layer "B.Cu")
-		(net "/3.3V")
-	)
-	(segment
-		(start 232.25 113.9)
-		(end 232.25 109.05)
-		(width 0.2)
-		(layer "B.Cu")
-		(net "/3.3V")
-	)
-	(segment
-		(start 229.75 110.099999)
-		(end 227.150001 107.5)
-		(width 0.2)
-		(layer "B.Cu")
-		(net "/Btn1")
-	)
-	(segment
-		(start 229.75 113.9)
-		(end 229.75 110.099999)
-		(width 0.2)
-		(layer "B.Cu")
-		(net "/Btn1")
-	)
-	(segment
 		(start 241.46 108.1)
 		(end 241.46 106.96)
@@
 		(net "Net-(R1-Pad2)")
 	)
+	(segment
+		(start 233.1 116.1)
+		(end 231.95 116.1)
+		(width 0.2)
+		(layer "B.Cu")
+		(net "/GND")
+	)
+	(segment
+		(start 231.95 116.1)
+		(end 229.75 113.9)
+		(width 0.2)
+		(layer "B.Cu")
+		(net "/GND")
+	)
+	(segment
+		(start 234.5 114.7)
+		(end 233.1 116.1)
+		(width 0.2)
+		(layer "B.Cu")
+		(net "/GND")
+	)
+	(segment
+		(start 234.5 111.3)
+		(end 234.5 114.7)
+		(width 0.2)
+		(layer "B.Cu")
+		(net "/GND")
+	)
+	(segment
+		(start 231.3 108.1)
+		(end 234.5 111.3)
+		(width 0.2)
+		(layer "B.Cu")
+		(net "/GND")
+	)
+	(segment
+		(start 232.25 112.599999)
+		(end 227.150001 107.5)
+		(width 0.2)
+		(layer "B.Cu")
+		(net "/BtnPower")
+	)
+	(segment
+		(start 232.25 113.9)
+		(end 232.25 112.599999)
+		(width 0.2)
+		(layer "B.Cu")
+		(net "/BtnPower")
+	)
 	(embedded_fonts no)
