File: kicad/rpi_hat/rpi_hat/rpi_hat.kicad_pcb (KiCad board)
At the start: 2 copper layers, 65 x 56 mm, 15 parts, among them J1 FrontButtons, J2 PowerButton, J3 PowerWakeup, J4 DisplaySPI, J5 BatteryLevel, J6 GPIO

Commit message: add power switch to it8951
Parts:
- removed C1: 0.1uF, Capacitor_THT:C_Disc_D10.0mm_W2.5mm_P5.00mm
- removed C2: 10uF, Capacitor_THT:C_Disc_D10.0mm_W2.5mm_P5.00mm
- removed C3: 220nF, Capacitor_THT:C_Radial_D8.0mm_H7.0mm_P3.50mm
- added Q1: AO3401A, Package_TO_SOT_SMD:SOT-23, F.Cu at (147.6, 74.0)
- added Q2: PN2222A, Package_TO_SOT_THT:TO-92_Inline, F.Cu at (147.5, 65.9)
- added R3: 10k, Resistor_THT:R_Axial_DIN0207_L6.3mm_D2.5mm_P10.16mm_Horizontal, F.Cu at (152.5, 67.2)
- added R4: 10k, Resistor_THT:R_Axial_DIN0207_L6.3mm_D2.5mm_P10.16mm_Horizontal, F.Cu at (147.8, 62.8)
Connections:
- J4 pad 1: +5V -> /SPI_PWR
Routing:
- net /SPI_PWR: track 0.00 -> 36.2 mm
- net +5V: track 103.4 -> 118.0 mm
- net Net-(Q1-G): track 0.00 -> 12.0 mm
- net /GPIO12/PWM0: track 0.00 -> 6.96 mm
- net Net-(Q2-B): track 0.00 -> 6.20 mm
- net /GPIO8/SPI0.CE0: track 39.9 -> 39.4 mm

Commit message: fix bug in power on button routing in hat
Connections:
- J2 pad 1: +3V3 -> /BtnPower
- J2 pad 2: /BtnPower -> GND
- J3 pad 1: unconnected-(J3-Pin_1-Pad1) -> /BtnPower
- J3 pad 2: /BtnPower -> unconnected-(J3-Pin_2-Pad2)
Routing:
- net +3V3: track 79.8 -> 69.9 mm
- net /BtnPower: track 47.7 -> 40.1 mm

Commit message: wip
Parts:
- added R5: 10k, Resistor_THT:R_Axial_DIN0207_L6.3mm_D2.5mm_P10.16mm_Horizontal, F.Cu at (119.3, 56.7)
Connections:
- J3 pad 1: /BtnPower -> Net-(J3-Pin_1)
- J5 pad 1: /BatteryPwr -> unconnected-(J5-Pin_1-Pad1)
- J5 pad 3: unconnected-(J5-Pin_3-Pad3) -> /BatteryPwr
Routing:
- net /BtnPower: track 40.1 -> 55.0 mm
- net Net-(J3-Pin_1): track 0.00 -> 3.10 mm
- net /BatteryPwr: track 4.45 -> 6.90 mm
