File: kicad/rpi_hat/rpi_hat/rpi_hat.kicad_pcb (KiCad board)
At the start: 2 copper layers, 65 x 56 mm, 16 parts, among them J1 FrontButtons, J2 PowerButton, J3 PowerWakeup, J4 DisplaySPI, J5 BatteryLevel, J6 GPIO, Q1 AO3401A, Q2 PN2222A

Commit message: add script to read voltage from adc and fix hat
Connections:
- J5 pad 1: /BatteryPwr -> unconnected-(J5-Pin_1-Pad1)
- J5 pad 3: unconnected-(J5-Pin_3-Pad3) -> /BatteryPwr
Routing:
- net /BatteryPwr: track 4.45 -> 7.16 mm
Changed lines of the file:
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@@
 			(remove_unused_layers no)
 			(roundrect_rratio 0.147059)
-			(net "/BatteryPwr")
+			(net "unconnected-(J5-Pin_1-Pad1)")
 			(pinfunction "Pin_1_1")
-			(pintype "passive")
+			(pintype "passive+no_connect")
 		)
 		(pad "2" thru_hole oval
@@
 			(layers "*.Cu" "*.Mask")
 			(remove_unused_layers no)
-			(net "unconnected-(J5-Pin_3-Pad3)")
+			(net "/BatteryPwr")
 			(pinfunction "Pin_3_3")
-			(pintype "passive+no_connect")
+			(pintype "passive")
 		)
 		(pad "4" thru_hole oval
@@
 	(segment
 		(start 119.83 74.28)
-		(end 115.38 74.28)
-		(width 0.2)
-		(layer "F.Cu")
+		(end 117.9 76.21)
+		(width 0.2)
+		(layer "F.Cu")
+		(net "/BatteryPwr")
+	)
+	(segment
+		(start 115.78 79.32)
+		(end 115.34 79.32)
+		(width 0.2)
+		(layer "F.Cu")
+		(net "/BatteryPwr")
+	)
+	(segment
+		(start 117.9 77.2)
+		(end 115.78 79.32)
+		(width 0.2)
+		(layer "F.Cu")
+		(net "/BatteryPwr")
+	)
+	(segment
+		(start 117.9 76.21)
+		(end 117.9 77.2)
+		(width 0.2)
+		(layer "F.Cu")

Commit message: wip
Parts:
- added R5: 10k, Resistor_THT:R_Axial_DIN0207_L6.3mm_D2.5mm_P10.16mm_Horizontal, F.Cu at (119.3, 56.8)
Connections:
- J2 pad 1: +3V3 -> /BtnPower
- J2 pad 2: /BtnPower -> GND
- J3 pad 1: unconnected-(J3-Pin_1-Pad1) -> Net-(J3-Pin_1)
- J3 pad 2: /BtnPower -> unconnected-(J3-Pin_2-Pad2)
Routing:
- net +3V3: track 79.8 -> 69.9 mm
- net /BtnPower: track 47.7 -> 53.7 mm
- net Net-(J3-Pin_1): track 0.00 -> 4.16 mm

Commit message: finish battery support
Connections:
- J5 pad 4: GND -> /BatterNNP16
- J6 pad 33: GND -> /BatterNNP16
- R2 pad 1: GND -> /BatterNNP16
Routing:
- net /BatterNNP16: track 0.00 -> 120.4 mm
- net +3V3: track 69.9 -> 72.0 mm
- net +5V: track 118.0 -> 119.4 mm
