File: kicad/rpi_hat/rpi_hat/rpi_hat.kicad_pcb (KiCad board)
At the start: 2 copper layers, 65 x 56 mm, 16 parts, among them J1 FrontButtons, J2 PowerButton, J3 PowerWakeup, J4 DisplaySPI, J5 BatteryLevel, J6 GPIO, Q1 AO3401A, Q2 PN2222A

Commit message: Add support for power on button (#8)
* add power button

* fix bug in power on button routing in hat

* update test_buttons.py script

* implement power off buttton in all fsm

* refactor display subsystem
Parts:
- added R5: 10k, Resistor_THT:R_Axial_DIN0207_L6.3mm_D2.5mm_P10.16mm_Horizontal, F.Cu at (119.3, 56.7)
Connections:
- J2 pad 1: +3V3 -> /BtnPower
- J2 pad 2: /BtnPower -> GND
- J3 pad 1: unconnected-(J3-Pin_1-Pad1) -> Net-(J3-Pin_1)
- J3 pad 2: /BtnPower -> unconnected-(J3-Pin_2-Pad2)
- J5 pad 1: /BatteryPwr -> unconnected-(J5-Pin_1-Pad1)
- J5 pad 3: unconnected-(J5-Pin_3-Pad3) -> /BatteryPwr
Routing:
- net Net-(Q1-G): track 12.0 -> 24.1 mm
- net +3V3: track 79.8 -> 69.9 mm
- net /BtnPower: track 47.7 -> 55.0 mm
- net Net-(J3-Pin_1): track 0.00 -> 3.10 mm
- net /BatteryPwr: track 4.45 -> 6.90 mm

Commit message: Add support for battery (#10)
* add program to read voltage from adc and fix hat

* add battery support in lvgl
Parts:
- moved R5 0.10 mm to (119.3, 56.8)
Connections:
- J5 pad 4: GND -> /BatterNNP16
- J6 pad 33: GND -> /BatterNNP16
- R2 pad 1: GND -> /BatterNNP16
Routing:
- net /BatterNNP16: track 0.00 -> 120.4 mm
- net Net-(Q1-G): track 24.1 -> 12.0 mm
- net +3V3: track 69.9 -> 72.0 mm
- net +5V: track 118.0 -> 119.4 mm
- net /BtnPower: track 55.0 -> 53.7 mm
- net Net-(J3-Pin_1): track 3.10 -> 4.16 mm
